File: buck/buck/buck.kicad_pcb (KiCad board)
At the start: 2 copper layers, 51.1 x 24.6 mm, 32 parts, among them M1 CSD19537Q3, M2 CSD19537Q3, U1 LM5146RGYR

Commit message: PCB updates
Parts:
- removed G***: LOGO, OneTouch_Logo:onetouchlogo
- removed H1, H2, H3: MountingHole_Pad, TestPoint:TestPoint_Pad_4.0x7.4mm
- removed H6: MountingHole, MountingHole:MountingHole_2.2mm_M2_DIN965_Pad
- added C11: 560pF, Capacitor_SMD:C_0402_1005Metric, F.Cu at (113.2, 79.3)
- added C12: 22µF x 2, Capacitor_SMD:C_1206_3216Metric, F.Cu at (112.1, 85.5)
- added C13: 22µF x 2, Capacitor_SMD:C_1206_3216Metric, F.Cu at (111.0, 81.7)
- added J1: Conn_01x02_Socket, Connector_JST:JST_XH_S2B-XH-A_1x02_P2.50mm_Horizontal, F.Cu at (109.1, 90.0)
- C1: footprint Capacitor_SMD:C_1210_3225Metric -> Capacitor_SMD:C_1206_3216Metric
- C10: value 22µF x 2 -> 680pF; footprint Capacitor_SMD:C_1210_3225Metric -> Resistor_SMD:R_0402_1005Metric
- C2: value 58nF -> 2.2uF x 3; footprint Capacitor_SMD:C_0402_1005Metric -> Capacitor_SMD:C_1206_3216Metric
- C3: value 2.2µF -> 2.2uF x 3; footprint Capacitor_SMD:C_0402_1005Metric -> Capacitor_SMD:C_1206_3216Metric
- C4: value 100nF -> 56nF; footprint Capacitor_SMD:C_0603_1608Metric -> Capacitor_SMD:C_0402_1005Metric
- C5: value 3pF -> 2.2µF; footprint Capacitor_SMD:C_0805_2012Metric -> Capacitor_SMD:C_1206_3216Metric
- C6: footprint Capacitor_SMD:C_0603_1608Metric -> Capacitor_SMD:C_1210_3225Metric
- C7: value 8.2nF -> 3pF; footprint Resistor_SMD:R_0402_1005Metric -> Capacitor_SMD:C_0402_1005Metric
- C8: value 680pF -> 100nF; footprint Resistor_SMD:R_0402_1005Metric -> Capacitor_SMD:C_1210_3225Metric
- C9: value 580pF -> 8.2nF; footprint Capacitor_SMD:C_0402_1005Metric -> Resistor_SMD:R_0402_1005Metric
- H4: value MountingHole_Pad -> MountingHole; footprint TestPoint:TestPoint_Pad_4.0x7.4mm -> MountingHole:MountingHole_2.2mm_M2_DIN965_Pad
- R4: footprint Resistor_SMD:R_0603_1608Metric -> Resistor_SMD:R_1206_3216Metric
- R7: footprint Resistor_SMD:R_0805_2012Metric -> Resistor_SMD:R_0603_1608Metric
- R9: footprint Resistor_SMD:R_0603_1608Metric -> Resistor_SMD:R_0402_1005Metric
- moved H5 47.7 mm to (143.5, 99.1)
- moved H4 25.5 mm to (143.6, 94.0)
- moved C8 22.0 mm to (129.2, 80.2)
- moved C2 20.9 mm to (125.6, 72.7), turned to 0 degrees
- moved L1 19.1 mm to (122.9, 91.4), turned to 0 degrees
- moved R3 14.5 mm to (118.3, 69.6)
- moved C5 12.7 mm to (121.2, 78.8)
- moved C7 12.0 mm to (117.7, 79.1)
- moved C3 11.5 mm to (121.2, 74.1)
- moved R4 10.7 mm to (125.6, 70.3), turned to 0 degrees
- moved R6 10.3 mm to (118.3, 82.0), turned to 180 degrees
- moved C1 10.2 mm to (129.6, 75.2)
- moved U1 9.20 mm to (117.7, 76.1)
- moved M1 9.09 mm to (125.2, 80.4)
- moved R5 8.88 mm to (115.2, 82.0), turned to 180 degrees
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Connections:
- C10 pad 1: +7.4V -> Net-(U1-COMP)
- C10 pad 2: GND -> Net-(U1-FB)
- C2 pad 1: Net-(U1-SS_TRK) -> +BATT
- C3 pad 1: Net-(U1-VCC) -> +BATT
- C4 pad 1: Net-(U1-VIN) -> Net-(U1-SS_TRK)
- C5 pad 1: Net-(U1-ILIM) -> Net-(U1-VCC)
- C6 pad 1: Net-(U1-BST) -> Net-(U1-VIN)
- C6 pad 2: Net-(M1-D) -> GND
- C7 pad 1: Net-(U1-COMP) -> Net-(U1-ILIM)
- C7 pad 2: Net-(C7-Pad2) -> GND
- C8 pad 1: Net-(U1-COMP) -> Net-(U1-BST)
- C8 pad 2: Net-(U1-FB) -> Net-(M1-D)
- C9 pad 1: Net-(C9-Pad1) -> Net-(U1-COMP)
- C9 pad 2: Net-(U1-FB) -> Net-(C9-Pad2)
- H4 pad 1: GND -> (no net)
- R11 pad 2: Net-(C9-Pad1) -> Net-(C11-Pad1)
- R8 pad 1: Net-(C7-Pad2) -> Net-(C9-Pad2)
Routing:
- net Net-(M1-D): track 22.4 -> 0.00 mm
- net Net-(M2-G): track 11.9 -> 0.00 mm
- net Net-(U1-FB): track 11.0 -> 0.00 mm
- net Net-(U1-EN_UVLO): track 7.97 -> 0.00 mm
- net Net-(U1-VIN): track 7.34 -> 0.00 mm
- net Net-(U1-VCC): track 9.11 -> 2.02 mm
- net Net-(M1-G): track 6.30 -> 0.00 mm
- net Net-(U1-ILIM): track 4.38 -> 0.00 mm
- net Net-(U1-SYNCIN): track 3.49 -> 0.00 mm
- net Net-(U1-SS_TRK): track 2.48 -> 0.00 mm
- net Net-(C7-Pad2): track 2.42 -> 0.00 mm
- net Net-(U1-RT): track 2.32 -> 0.00 mm
- net Net-(U1-COMP): track 2.25 -> 0.00 mm
- net Net-(U1-PGOOD): track 1.77 -> 0.00 mm
- net Net-(U1-BST): track 1.70 -> 0.00 mm
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- removed copper zone on F.Cu, net +7.4V
- removed copper zone on F.Cu, net +BATT
- removed copper zone on F.Cu, net Net-(M1-D)
Other:
- board size 51.1 x 24.6 mm -> 25.3 x 31.7 mm
- board text removed: "GND"
